File: KiCad/Mini8085.kicad_pcb (KiCad board)
At the start: 2 copper layers, 100 x 80 mm, 45 parts, among them P1 POWER, P2 SIO, P3 SERIAL, P4 EXTENSION, P5 VBAT, SW1 RESET, U1 80C85A, U2 82C51A, U3 27C128, U4 62256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

Commit message: * Add Mini8085 - Board - 1.0.pdf * Update KiCad project to KiCad v6
Parts:
- removed G***: OSHW-logo_silkscreen-front_10mm, OSHW-logo:OSHW-logo_silkscreen-front_10mm
Connections:
- net /IO/~M renamed /IO/~{M}
- net /~CTS renamed /~{CTS}
- net /~INTA renamed /~{INTA}
- net /~RAM_CS renamed /~{RAM_CS}
- net /~RAM_CSO renamed /~{RAM_CSO}
- net /~RD renamed /~{RD}
- net /~ROM_CS renamed /~{ROM_CS}
- net /~RTS renamed /~{RTS}
- net /~SWAP_MEM renamed /~{SWAP_MEM}
- net /~USART_CS renamed /~{USART_CS}
- net /~WR renamed /~{WR}
- P3 pad 1: Net-(P3-Pad1) -> unconnected-(P3-Pad1)
- P3 pad 4: Net-(P3-Pad4) -> unconnected-(P3-Pad4)
- P3 pad 6: Net-(P3-Pad6) -> unconnected-(P3-Pad6)
- P3 pad 9: Net-(P3-Pad9) -> unconnected-(P3-Pad9)
- P3 pad GND: GND -> (no net)
- U1 pad 29: Net-(U1-Pad29) -> unconnected-(U1-Pad29)
- U1 pad 33: Net-(U1-Pad33) -> unconnected-(U1-Pad33)
- U1 pad 38: Net-(U1-Pad38) -> unconnected-(U1-Pad38)
- U2 pad 15: Net-(U2-Pad15) -> unconnected-(U2-Pad15)
- U2 pad 16: Net-(U2-Pad16) -> unconnected-(U2-Pad16)
- U2 pad 18: Net-(U2-Pad18) -> unconnected-(U2-Pad18)
Other:
- net class Default removed
- net class Power removed
- board text added: "IO/~{M}"
- board text added: "~{INTA}"
- board text added: "~{RD}"
- board text added: "~{SWAP_MEM}"
- board text added: "~{WR}"
- board text removed: "IO/~M"
- board text removed: "~INTA"
- board text removed: "~RD"
- board text removed: "~SWAP_MEM"
- board text removed: "~WR"
